File: macropad/macropad.kicad_pcb (KiCad board)
At the start: 2 copper layers, 97 parts, among them J1 USB_C_Receptacle_USB2.0_14P, SW1 SW_SPST, SW10 SW_SPST, SW11 SW_SPST, SW12 SW_SPST, SW13 SW_SPST, SW14 SW_SPST, SW15 SW_SPST, SW16 SW_SPST, SW17 SW_SPST, SW18 SW_SPST, SW19 SW_SPST, SW2 SW_SPST, SW20 SW_SPST, SW21 SW_SPST, SW22 SW_SPST, SW23 SW_SPST, SW24 SW_SPST, SW25 SW_SPST, SW26 SW_SPST, SW27 SW_SPST, SW28 SW_SPST, SW29 SW_SPST, SW3 SW_SPST, SW30 SW_SPST, SW31 SW_SPST, SW32 SW_SPST, SW33 SW_SPST, SW34 SW_SPST, SW35 SW_SPST, SW36 SW_SPST, SW37 SW_SPST, SW38 SW_SPST, SW39 SW_SPST, SW4 SW_SPST, SW40 SW_SPST, SW41 SW_Push, SW5 SW_SPST, SW6 SW_SPST, SW7 SW_SPST, SW8 SW_SPST, SW9 SW_SPST, U1 ATmega32U4-A, Y1 Crystal_GND24_Small

Commit message: a
Parts:
- added J2: AVR-ISP-6, Connector_IDC:IDC-Header_2x03_P2.54mm_Vertical, F.Cu at (99.8, 79.0)
- J1, R2, R3, R5, R6: moved to F.Cu
- moved R6 32.4 mm to (84.5, 76.1), turned to 180 degrees
- moved R3 25.5 mm to (84.5, 79.3)
- moved J1 23.4 mm to (71.8, 80.3), turned to -90 degrees
- moved R2 21.7 mm to (84.5, 81.2)
- moved R5 15.7 mm to (84.5, 84.3), turned to 180 degrees
Connections:
- net DU+ renamed UD+
- net DU- renamed UD-
- J1 pad A4: Net-(J1-VBUS-PadA4) -> +5V
- J1 pad B4: Net-(J1-VBUS-PadA4) -> +5V
- U1 pad 10: ROW2 -> MOSI
- U1 pad 11: ROW3 -> MISO
- U1 pad 12: ROW4 -> unconnected-(U1-PB7-Pad12)
- U1 pad 18: COL1 -> unconnected-(U1-PD0-Pad18)
- U1 pad 19: COL2 -> unconnected-(U1-PD1-Pad19)
- U1 pad 20: COL3 -> unconnected-(U1-PD2-Pad20)
- U1 pad 21: COL4 -> unconnected-(U1-PD3-Pad21)
- U1 pad 22: COL5 -> unconnected-(U1-PD5-Pad22)
- U1 pad 26: COL6 -> unconnected-(U1-PD6-Pad26)
- U1 pad 27: COL7 -> unconnected-(U1-PD7-Pad27)
- U1 pad 28: COL8 -> unconnected-(U1-PB4-Pad28)
- U1 pad 29: COL9 -> unconnected-(U1-PB5-Pad29)
- U1 pad 30: COL10 -> unconnected-(U1-PB6-Pad30)
- U1 pad 8: unconnected-(U1-PB0-Pad8) -> SS
- U1 pad 9: ROW1 -> SCK
Routing:
- net ROW4: track 89.7 -> 0.00 mm, vias 2 -> 0
- net ROW3: track 67.8 -> 0.00 mm, vias 2 -> 0
- net ROW2: track 51.5 -> 0.00 mm, vias 2 -> 0
- net +5V: track 67.4 -> 102.9 mm, vias 5 -> 7
- net GND: track 114.2 -> 95.8 mm
- net ROW1: track 13.2 -> 0.00 mm
- net UD-: track 21.1 -> 33.4 mm, vias 0 -> 1
- net UD+: track 21.4 -> 32.4 mm, vias 0 -> 1
- net D+: track 10.2 -> 12.8 mm
- net D-: track 10.8 -> 11.6 mm
- net Net-(J1-CC2): track 8.02 -> 7.24 mm
- net Net-(J1-CC1): track 8.31 -> 7.56 mm
