File: macropad/macropad.kicad_sch (KiCad schematic)
At the start: 97 parts, among them J1 USB_C_Receptacle_USB2.0_14P, SW1 SW_SPST, SW10 SW_SPST, SW11 SW_SPST, SW12 SW_SPST, SW13 SW_SPST, SW14 SW_SPST, SW15 SW_SPST, SW16 SW_SPST, SW17 SW_SPST, SW18 SW_SPST, SW19 SW_SPST, SW2 SW_SPST, SW20 SW_SPST, SW21 SW_SPST, SW22 SW_SPST, SW23 SW_SPST, SW24 SW_SPST, SW25 SW_SPST, SW26 SW_SPST, SW27 SW_SPST, SW28 SW_SPST, SW29 SW_SPST, SW3 SW_SPST, SW30 SW_SPST, SW31 SW_SPST, SW32 SW_SPST, SW33 SW_SPST, SW34 SW_SPST, SW35 SW_SPST, SW36 SW_SPST, SW37 SW_SPST, SW38 SW_SPST, SW39 SW_SPST, SW4 SW_SPST, SW40 SW_SPST, SW41 SW_Push, SW5 SW_SPST, SW6 SW_SPST, SW7 SW_SPST, SW8 SW_SPST, SW9 SW_SPST, U1 ATmega32U4-A, Y1 Crystal_GND24_Small

Commit message: a
Parts:
- added J2: AVR-ISP-6, Connector_IDC:IDC-Header_2x03_P2.54mm_Vertical, symbol Connector:AVR-ISP-6
Connections:
- net +5V: now also J1.A4 (VBUS), J1.A9 (VBUS), J1.B4 (VBUS), J1.B9 (VBUS), J2.2 (VCC)
- net GND: now also J2.6 (GND)
- net MOSI: now reaches U1.10 (PB2)
- net MOSI: now also J2.4 (MOSI)
- net MISO: now reaches U1.11 (PB3)
- net MISO: now also J2.1 (MISO)
- net UD-: now reaches R3.1, U1.3 (D-)
- net UD+: now reaches R2.2, U1.4 (D+)
- net SS: now reaches U1.8 (PB0)
- net SS: now also J2.5 (~{RST})
- net SCK: now reaches U1.9 (PB1)
- net SCK: now also J2.3 (SCK)

Commit message: aaaa mx
Parts:
- added H1, H2, H3, H4, H5: MountingHole, MountingHole:MountingHole_5.3mm_M5, symbol Mechanical:MountingHole
- J1: footprint Type-C:HRO-TYPE-C-31-M-13 -> Connector_USB:USB_C_Receptacle_HRO_TYPE-C-31-M-12
Connections:
- net COL1: now also U1.41 (PF0)
- net COL10: now also U1.22 (PD5)
- net COL2: now also U1.40 (PF1)
- net COL3: now also U1.39 (PF4)
- net COL4: now also U1.38 (PF5)
- net COL5: now also U1.28 (PB4)
- net COL6: now also U1.27 (PD7)
- net COL7: now also U1.26 (PD6)
- net COL8: now also U1.25 (PD4)
- net COL9: now also U1.21 (PD3)
- net ROW1: now also U1.12 (PB7)
- net ROW2: now also U1.29 (PB5)
- net ROW3: now also U1.30 (PB6)
- net ROW4: now also U1.31 (PC6)
